Commit message: undo submodules commits - should no longer be any submodules

File: scenes/hubo-models/hubosimple.urdf (robot description, URDF)
Before this commit: robot jaemiHubo, 66 links, 65 joints
Links:
- link Body_LEP: geometry collision mesh filename=hubosimple-dae/Body_LEP_col.dae; visual mesh filename=hubosimple-dae/Body_LEP_vis.dae
- link Body_LSP: geometry collision mesh filename=hubosimple-dae/Body_LSP_col.dae; visual mesh filename=hubosimple-dae/Body_LSP_vis.dae
- link Body_LSR: geometry collision mesh filename=hubosimple-dae/Body_LSR_col.dae; visual mesh filename=hubosimple-dae/Body_LSR_vis.dae
- link Body_LSY: geometry collision mesh filename=hubosimple-dae/Body_LSY_col.dae; visual mesh filename=hubosimple-dae/Body_LSY_vis.dae
- link Body_LWY: geometry collision mesh filename=hubosimple-dae/Body_LWY_col.dae; visual mesh filename=hubosimple-dae/Body_LWY_vis.dae
- link Body_REP: geometry collision mesh filename=hubosimple-dae/Body_REP_col.dae; visual mesh filename=hubosimple-dae/Body_REP_vis.dae
- link Body_RSP: geometry collision mesh filename=hubosimple-dae/Body_RSP_col.dae; visual mesh filename=hubosimple-dae/Body_RSP_vis.dae
- link Body_RSR: geometry collision mesh filename=hubosimple-dae/Body_RSR_col.dae; visual mesh filename=hubosimple-dae/Body_RSR_vis.dae
- link Body_RSY: geometry collision mesh filename=hubosimple-dae/Body_RSY_col.dae; visual mesh filename=hubosimple-dae/Body_RSY_vis.dae
- link Body_RWY: geometry collision mesh filename=hubosimple-dae/Body_RWY_col.dae; visual mesh filename=hubosimple-dae/Body_RWY_vis.dae
- link Head: geometry collision mesh filename=hubosimple-dae/Head_col.dae; visual mesh filename=hubosimple-dae/Head_vis.dae
- link HeadYaw: geometry visual mesh filename=hubosimple-dae/HeadYaw_vis.dae
- link Hip: geometry collision mesh filename=hubosimple-dae/Hip_col.dae; visual mesh filename=hubosimple-dae/Hip_vis.dae
- link Torso: geometry collision mesh filename=hubosimple-dae/Torso_col.dae; visual mesh filename=hubosimple-dae/Torso_vis.dae
- link leftAnklePitch: geometry collision mesh filename=hubosimple-dae/leftAnklePitch_col.dae; visual mesh filename=hubosimple-dae/leftAnklePitch_vis.dae
- link leftFoot: geometry collision mesh filename=hubosimple-dae/leftFoot_col.dae; visual mesh filename=hubosimple-dae/leftFoot_vis.dae
- link leftHip: geometry collision mesh filename=hubosimple-dae/leftHip_col.dae; visual mesh filename=hubosimple-dae/leftHip_vis.dae
- link leftHipPitchRoll: geometry collision mesh filename=hubosimple-dae/leftHipPitchRoll_col.dae; visual mesh filename=hubosimple-dae/leftHipPitchRoll_vis.dae
- link leftIndexDistal: geometry visual mesh filename=hubosimple-dae/leftIndexDistal_vis.dae
- link leftIndexMedial: geometry visual mesh filename=hubosimple-dae/leftIndexMedial_vis.dae
- link leftIndexProximal: geometry visual mesh filename=hubosimple-dae/leftIndexProximal_vis.dae
- link leftKneeLower: geometry collision mesh filename=hubosimple-dae/leftKneeLower_col.dae; visual mesh filename=hubosimple-dae/leftKneeLower_vis.dae
- link leftKneeUpper: geometry collision mesh filename=hubosimple-dae/leftKneeUpper_col.dae; visual mesh filename=hubosimple-dae/leftKneeUpper_vis.dae
- link leftMiddleDistal: geometry visual mesh filename=hubosimple-dae/leftMiddleDistal_vis.dae
- link leftMiddleMedial: geometry visual mesh filename=hubosimple-dae/leftMiddleMedial_vis.dae
- link leftMiddleProximal: geometry visual mesh filename=hubosimple-dae/leftMiddleProximal_vis.dae
- link leftPalm: geometry visual mesh filename=hubosimple-dae/leftPalm_vis.dae
- link leftPinkyDistal: geometry visual mesh filename=hubosimple-dae/leftPinkyDistal_vis.dae
- link leftPinkyMedial: geometry visual mesh filename=hubosimple-dae/leftPinkyMedial_vis.dae
- link leftPinkyProximal: geometry visual mesh filename=hubosimple-dae/leftPinkyProximal_vis.dae
- link leftRingDistal: geometry visual mesh filename=hubosimple-dae/leftRingDistal_vis.dae
- link leftRingMedial: geometry visual mesh filename=hubosimple-dae/leftRingMedial_vis.dae
- link leftRingProximal: geometry visual mesh filename=hubosimple-dae/leftRingProximal_vis.dae
- link leftThumbDistal: geometry visual mesh filename=hubosimple-dae/leftThumbDistal_vis.dae
- link leftThumbMedial: geometry visual mesh filename=hubosimple-dae/leftThumbMedial_vis.dae
- link leftThumbProximal: geometry visual mesh filename=hubosimple-dae/leftThumbProximal_vis.dae
- link leftUJoint: geometry collision mesh filename=hubosimple-dae/leftUJoint_col.dae; visual mesh filename=hubosimple-dae/leftUJoint_vis.dae
- link rightAnklePitch: geometry collision mesh filename=hubosimple-dae/rightAnklePitch_col.dae; visual mesh filename=hubosimple-dae/rightAnklePitch_vis.dae
- link rightFoot: geometry collision mesh filename=hubosimple-dae/rightFoot_col.dae; visual mesh filename=hubosimple-dae/rightFoot_vis.dae
- link rightHip: geometry collision mesh filename=hubosimple-dae/rightHip_col.dae; visual mesh filename=hubosimple-dae/rightHip_vis.dae
- link rightHipPitchRoll: geometry collision mesh filename=hubosimple-dae/rightHipPitchRoll_col.dae; visual mesh filename=hubosimple-dae/rightHipPitchRoll_vis.dae
- link rightIndexDistal: geometry visual mesh filename=hubosimple-dae/rightIndexDistal_vis.dae
- link rightIndexMedial: geometry visual mesh filename=hubosimple-dae/rightIndexMedial_vis.dae
- link rightIndexProximal: geometry visual mesh filename=hubosimple-dae/rightIndexProximal_vis.dae
- link rightKneeLower: geometry collision mesh filename=hubosimple-dae/rightKneeLower_col.dae; visual mesh filename=hubosimple-dae/rightKneeLower_vis.dae
- link rightKneeUpper: geometry collision mesh filename=hubosimple-dae/rightKneeUpper_col.dae; visual mesh filename=hubosimple-dae/rightKneeUpper_vis.dae
- link rightMiddleDistal: geometry visual mesh filename=hubosimple-dae/rightMiddleDistal_vis.dae
- link rightMiddleMedial: geometry visual mesh filename=hubosimple-dae/rightMiddleMedial_vis.dae
- link rightMiddleProximal: geometry visual mesh filename=hubosimple-dae/rightMiddleProximal_vis.dae
- link rightPalm: geometry visual mesh filename=hubosimple-dae/rightPalm_vis.dae
- link rightPinkyDistal: geometry visual mesh filename=hubosimple-dae/rightPinkyDistal_vis.dae
- link rightPinkyMedial: geometry visual mesh filename=hubosimple-dae/rightPinkyMedial_vis.dae
- link rightPinkyProximal: geometry visual mesh filename=hubosimple-dae/rightPinkyProximal_vis.dae
- link rightRingDistal: geometry visual mesh filename=hubosimple-dae/rightRingDistal_vis.dae
- link rightRingMedial: geometry visual mesh filename=hubosimple-dae/rightRingMedial_vis.dae
- link rightRingProximal: geometry visual mesh filename=hubosimple-dae/rightRingProximal_vis.dae
- link rightThumbDistal: geometry visual mesh filename=hubosimple-dae/rightThumbDistal_vis.dae
- link rightThumbMedial: geometry visual mesh filename=hubosimple-dae/rightThumbMedial_vis.dae
- link rightThumbProximal: geometry visual mesh filename=hubosimple-dae/rightThumbProximal_vis.dae
- link rightUJoint: geometry collision mesh filename=hubosimple-dae/rightUJoint_col.dae; visual mesh filename=hubosimple-dae/rightUJoint_vis.dae
