Commit message: No need for .stl files; fixed urdf

File: scenes/driving_wheel_full.urdf (robot description, URDF)
Before this commit: robot valve, 2 links, 1 joints
Links:
- link base: geometry collision mesh filename=objects/logitech_driving_force_pro_wheel_base_small.3ds scale=0.025399986 0.025399986 0.025399986; visual mesh filename=objects/logitech_driving_force_pro_wheel_base_small.3ds scale=0.025399986 0.025399986 0.025399986
- link handle: geometry collision mesh filename=objects/logitech_driving_force_pro_wheel_small.3ds scale=0.025399986 0.025399986 0.025399986; visual mesh filename=objects/logitech_driving_force_pro_wheel_small.3ds scale=0.025399986 0.025399986 0.025399986

Commit message: Fixes to driving wheel urdfs

File: scenes/driving_wheel_full.urdf (robot description, URDF)
Before this commit: robot valve, 2 links, 1 joints
Links:
- link base: mass 1.0 -> 0.6

Commit message: Cleanup of driving wheel urdf

File: scenes/driving_wheel_full.urdf (robot description, URDF)
Before this commit: robot valve, 2 links, 1 joints
Joints:
- joint base_to_handle: origin xyz=0 0 0 rpy=0 -0.4 0 -> xyz=0 0 0 rpy=0 0 0

Commit message: Further cleanup of urdf models

File: scenes/driving_wheel_full.urdf (robot description, URDF)
Before this commit: robot valve, 2 links, 1 joints
Links:
- link base: mass 0.6 -> 10.0
